Commit message: mega commit

File: surfmotion_examples/kuka/iiwa_custom_description/urdf/iiwa_custom.urdf.xacro (robot description, xacro)
@@ -4,5 +4,5 @@
   <link name="world"/>
   <xacro:iiwa parent="world" prefix="">
-    <origin xyz="0 0 0" rpy="0 0 0"/>
+    <origin xyz="0.4 0 0" rpy="0 0 0"/>
   </xacro:iiwa>
 </robot>
